Commit message: Update rover_model.urdf

File: rover_model.urdf (robot description, URDF)
Before this commit: robot myfirst, 11 links, 2 joints
Joints:
- joint mount to arm: origin xyz=0.2 0.01 0 rpy=0 0 0 -> xyz=0 0 0 rpy=0 0 0

Commit message: Update rover_model.urdf

File: rover_model.urdf (robot description, URDF)
Before this commit: robot myfirst, 11 links, 2 joints
Links:
- added link /ff; visual box size=.01 .01 .01
- added link /fl; visual box size=.01 .01 .01
- added link /fr; visual box size=.01 .01 .01

Commit message: set it up as a proper ros package

File: rover_model.urdf (robot description, URDF)
Before this commit: robot myfirst, 14 links, 2 joints
Links:
- removed link /ff
- removed link /fl
- removed link /fr
- removed link base
- removed link head
- removed link mount
- added link base_link; visual box size=.6 .6 .3
- added link fcu; visual box size=.3 .2 .15
- added link ff; visual box size=.01 .01 .01
- added link fl; visual box size=.01 .01 .01
- added link fr; visual box size=.01 .01 .01
- added link mount1; visual box size=.02 .02 .2
- link mount3: geometry visual box size=.04 .04 .27
Joints:
- removed joint base_to_head
- added joint base_to_mount: type fixed, parent base_link, child mount1
- added joint base_to_neck: type fixed, parent base_link, child neck
- added joint base_to_wheel1: type fixed, parent base_link, child wheel1
- added joint base_to_wheel2: type fixed, parent base_link, child wheel2
- added joint base_to_wheel3: type fixed, parent base_link, child wheel3
- added joint base_to_wheel4: type fixed, parent base_link, child wheel4
- added joint mount_to_ff: type fixed, parent mount3, child ff
- added joint mount_to_fl: type fixed, parent mount3, child fl
- added joint mount_to_fr: type fixed, parent mount3, child fr
- added joint mount_to_vertical: type fixed, parent mount1, child mount2
- added joint neck_to_head: type fixed, parent neck, child fcu
- added joint vertical_to_t: type fixed, parent mount2, child mount3

Commit message: got range visualization working

File: rover_model.urdf (robot description, URDF)
Before this commit: robot myfirst, 14 links, 13 joints
Links:
- added link camera; visual box size=.05 .05 .05
Joints:
- added joint head_to_camera: type fixed, parent fcu, child camera, origin xyz=0 0 0.65 rpy=0 0 0
- joint mount_to_ff: origin (none) -> xyz=.37 0.1 0.3 rpy=1.55 0.1 0; parent mount3 -> base_link
- joint mount_to_fl: origin (none) -> xyz=.37 0.1 0.3 rpy=1.55 0.1 1; parent mount3 -> base_link
- joint mount_to_fr: origin (none) -> xyz=.37 0.1 0.3 rpy=1.55 0.1 -1; parent mount3 -> base_link

Commit message: rviz and kinect_aux stuff

File: rover_model.urdf (robot description, URDF)
Before this commit: robot myfirst, 15 links, 14 joints
Links:
- removed link camera
- added link camera_link; visual box size=.05 .05 .05
Joints:
- joint head_to_camera: child camera -> camera_link
