Commit message: .

File: tank_model.urdf (robot description, URDF)
Before this commit: robot pi_robot, 6 links, 5 joints
Links:
- removed link enclosure_link
- removed link left_track_drive_link
- removed link left_track_link
- removed link right_track_drive_link
- removed link right_track_link
- added link camera_link; visual box size=0.3 0.43 0.24
- added link laser_link; visual box size=0.3 0.43 0.24
Joints:
- removed joint enclosure_joint
- removed joint left_track_drive_joint
- removed joint left_track_joint
- removed joint right_track_drive_joint
- removed joint right_track_joint
- added joint camera_joint: type fixed, parent base_link, child camera_link
- added joint laser_joint: type fixed, parent base_link, child laser_link
